File: rasp/hardware/hardware.sch (KiCad schematic (older format))
At the start: 43 parts, among them J10 Conn_01x02_Male, J11 Conn_01x02_Male, J12 Conn_01x02_Male, J13 Conn_01x02_Male, J14 Conn_01x02_Male, J15 Conn_01x02_Male, J16 Conn_01x02_Male, J17 Conn_01x02_Male, J18 Conn_01x02_Male, J19 Conn_01x02_Male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

Commit message: Added diode
Parts:
- added D8: D_Schottky, Diode_SMD:D_SMB, symbol Device:D_Schottky
Connections:
- net +5V: now also D8.1 (K); no longer J4.15 (Pin_15), J4.16 (Pin_16)
- new net +5VP: D8.2 (A), J4.15 (Pin_15), J4.16 (Pin_16)
Changed lines of the file:
@@
 Wire Wire Line
 	1700 1050 1850 1050
-$Comp
-L power:+5V #PWR0106
-U 1 1 5EE2252F
-P 1000 850
-F 0 "#PWR0106" H 1000 700 50  0001 C CNN
-F 1 "+5V" V 1000 1050 50  0000 C CNN
-F 2 "" H 1000 850 50  0000 C CNN
-F 3 "" H 1000 850 50  0000 C CNN
-	1    1000 850
-	1    0    0    -1
-$EndComp
-$Comp
-L power:+5V #PWR0107
-U 1 1 5EE2270A
-P 2000 850
-F 0 "#PWR0107" H 2000 700 50  0001 C CNN
-F 1 "+5V" V 2000 1050 50  0000 C CNN
-F 2 "" H 2000 850 50  0000 C CNN
-F 3 "" H 2000 850 50  0000 C CNN
-	1    2000 850
-	1    0    0    -1
-$EndComp
 Wire Wire Line
 	1700 1650 2000 1650
@@
 Text GLabel 5350 2300 2    50   Input ~ 0
 A3
+$Comp
+L power:+5VP #PWR011
+U 1 1 5F99FD3D
+P 2000 850
+F 0 "#PWR011" H 2000 700 50  0001 C CNN
+F 1 "+5VP" H 2015 1023 50  0000 C CNN
+F 2 "" H 2000 850 50  0001 C CNN
+F 3 "" H 2000 850 50  0001 C CNN
+	1    2000 850
+	1    0    0    -1
+$EndComp
+$Comp
+L power:+5VP #PWR010
+U 1 1 5F99FF13
+P 1000 850
+F 0 "#PWR010" H 1000 700 50  0001 C CNN
+F 1 "+5VP" H 1015 1023 50  0000 C CNN
+F 2 "" H 1000 850 50  0001 C CNN
+F 3 "" H 1000 850 50  0001 C CNN
+	1    1000 850
+	1    0    0    -1
+$EndComp
+$Comp
+L Device:D_Schottky D8
+U 1 1 5F9A00B8
+P 3200 850
+F 0 "D8" H 3200 634 50  0000 C CNN
+F 1 "D_Schottky" H 3200 725 50  0000 C CNN
+F 2 "Diode_SMD:D_SMB" H 3200 850 50  0001 C CNN
+F 3 "~" H 3200 850 50  0001 C CNN
+	1    3200 850
+	-1   0    0    1
+$EndComp
+$Comp
+L power:+5VP #PWR03
+U 1 1 5F9A0284
+P 2750 750
+F 0 "#PWR03" H 2750 600 50  0001 C CNN
+F 1 "+5VP" H 2765 923 50  0000 C CNN
+F 2 "" H 2750 750 50  0001 C CNN
+F 3 "" H 2750 750 50  0001 C CNN
+	1    2750 750
+	1    0    0    -1
+$EndComp
+Wire Wire Line
+	3050 850  2750 850
+Wire Wire Line
+	2750 850  2750 750
+$Comp
+L power:+5V #PWR02
+U 1 1 5F9AF711
+P 3650 700
+F 0 "#PWR02" H 3650 550 50  0001 C CNN
+F 1 "+5V" H 3650 840 50  0000 C CNN
+F 2 "" H 3650 700 50  0000 C CNN
+F 3 "" H 3650 700 50  0000 C CNN
+	1    3650 700
+	1    0    0    -1
+$EndComp
+Wire Wire Line
+	3350 850  3650 850
+Wire Wire Line
+	3650 850  3650 700
 $EndSCHEMATC

Commit message: Added i2c connector
Parts:
- added J1: Conn_01x04_Male, Connector_PinHeader_2.54mm:PinHeader_1x04_P2.54mm_Horizontal, symbol Connector:Conn_01x04_Male
- added R12, R13: 2k2, Resistor_SMD:R_0805_2012Metric, symbol Device:R
- R10, R11, R3, R5, R8, R9: value 20K -> 18k
- R2: value R -> 820R
Connections:
- net +3V3: now also J1.4 (Pin_4), R12.1, R13.1
- net GND: now also J1.3 (Pin_3)
- net GPIO2(SDA1): now also J1.2 (Pin_2), R13.2
- net GPIO3(SCL1): now also J1.1 (Pin_1), R12.2
Other:
- moved on the sheet: D5, R2
Changed lines of the file:
@@
 U 1 1 5E6DCAD9
 P 1100 5850
-F 0 "J16" V 1253 5663 50  0000 R CNN
-F 1 "Conn_01x02_Male" V 1000 6300 50  0000 R CNN
+F 0 "J16" H 1253 5663 50  0000 R CNN
+F 1 "Conn_01x02_Male" V 1000 5850 50  0000 R CNN
 F 2 "Connector_PinHeader_2.54mm:PinHeader_1x02_P2.54mm_Vertical" H 1100 5850 50  0001 C CNN
 F 3 "~" H 1100 5850 50  0001 C CNN
@@
 L Device:R R2
 U 1 1 5EE3A0BC
-P 1000 3950
-F 0 "R2" H 1070 3996 50  0000 L CNN
-F 1 "R" H 1070 3905 50  0000 L CNN
-F 2 "Resistor_SMD:R_0805_2012Metric" V 930 3950 50  0001 C CNN
-F 3 "~" H 1000 3950 50  0001 C CNN
-	1    1000 3950
+P 800 3950
+F 0 "R2" H 870 3996 50  0000 L CNN
+F 1 "820R" H 870 3905 50  0000 L CNN
+F 2 "Resistor_SMD:R_0805_2012Metric" V 730 3950 50  0001 C CNN
+F 3 "~" H 800 3950 50  0001 C CNN
+	1    800  3950
 	1    0    0    -1
 $EndComp
@@
 L power:GND #PWR0114
 U 1 1 5EE3A180
-P 1000 4200
-F 0 "#PWR0114" H 1000 3950 50  0001 C CNN
-F 1 "GND" H 1000 4050 50  0000 C CNN
-F 2 "" H 1000 4200 50  0000 C CNN
-F 3 "" H 1000 4200 50  0000 C CNN
-	1    1000 4200
+P 800 4200
+F 0 "#PWR0114" H 800 3950 50  0001 C CNN
+F 1 "GND" H 800 4050 50  0000 C CNN
+F 2 "" H 800 4200 50  0000 C CNN
+F 3 "" H 800 4200 50  0000 C CNN
+	1    800  4200
 	1    0    0    -1
 $EndComp
@@
 L Device:LED D5
 U 1 1 5EE3A374
-P 1000 3550
-F 0 "D5" V 1038 3433 50  0000 R CNN
-F 1 "LED" V 947 3433 50  0000 R CNN
-F 2 "LED_SMD:LED_0805_2012Metric" H 1000 3550 50  0001 C CNN
-F 3 "~" H 1000 3550 50  0001 C CNN
-	1    1000 3550
-	0    -1   -1   0
-$EndComp
-Wire Wire Line
-	1000 3700 1000 3800
-Wire Wire Line
-	1000 4100 1000 4200
+P 800 3550
+F 0 "D5" V 838 3433 50  0000 R CNN
+F 1 "LED" V 747 3433 50  0000 R CNN
+F 2 "LED_SMD:LED_0805_2012Metric" H 800 3550 50  0001 C CNN
+F 3 "~" H 800 3550 50  0001 C CNN
+	1    800  3550
+	0    -1   -1   0
+$EndComp
+Wire Wire Line
+	800  3700 800  3800
+Wire Wire Line
+	800  4100 800  4200
 Text Notes 7000 6750 0    50   ~ 0
 SHIELD EXP430FR2355 PARA CARRINHO AUTÔNOMO\nLIGAÇÃO CONFORME PLACA DE POTÊNCIA
@@
 P 3400 5700
 F 0 "R9" H 3470 5746 50  0000 L CNN
-F 1 "20K" H 3470 5655 50  0000 L CNN
+F 1 "18k" H 3470 5655 50  0000 L CNN
 F 2 "Resistor_SMD:R_0805_2012Metric" V 3330 5700 50  0001 C CNN
 F 3 "~" H 3400 5700 50  0001 C CNN
@@
 P 1450 5700
 F 0 "R8" H 1520 5746 50  0000 L CNN
-F 1 "20K" H 1520 5655 50  0000 L CNN
+F 1 "18k" H 1520 5655 50  0000 L CNN
 F 2 "Resistor_SMD:R_0805_2012Metric" V 1380 5700 50  0001 C CNN
 F 3 "~" H 1450 5700 50  0001 C CNN
@@
 P 5650 3650
 F 0 "R3" H 5720 3696 50  0000 L CNN
-F 1 "20K" H 5720 3605 50  0000 L CNN
+F 1 "18k" H 5720 3605 50  0000 L CNN
 F 2 "Resistor_SMD:R_0805_2012Metric" V 5580 3650 50  0001 C CNN
 F 3 "~" H 5650 3650 50  0001 C CNN
@@
 P 5650 4750
 F 0 "R5" H 5720 4796 50  0000 L CNN
-F 1 "20K" H 5720 4705 50  0000 L CNN
+F 1 "18k" H 5720 4705 50  0000 L CNN
 F 2 "Resistor_SMD:R_0805_2012Metric" V 5580 4750 50  0001 C CNN
 F 3 "~" H 5650 4750 50  0001 C CNN
@@
 P 5650 5950
 F 0 "R10" H 5720 5996 50  0000 L CNN
-F 1 "20K" H 5720 5905 50  0000 L CNN
+F 1 "18k" H 5720 5905 50  0000 L CNN
 F 2 "Resistor_SMD:R_0805_2012Metric" V 5580 5950 50  0001 C CNN
 F 3 "~" H 5650 5950 50  0001 C CNN
@@
 P 7100 6000
 F 0 "R11" H 7170 6046 50  0000 L CNN
-F 1 "20K" H 7170 5955 50  0000 L CNN
+F 1 "18k" H 7170 5955 50  0000 L CNN
 F 2 "Resistor_SMD:R_0805_2012Metric" V 7030 6000 50  0001 C CNN
 F 3 "~" H 7100 6000 50  0001 C CNN
@@
 L power:+3.3V #PWR0136
 U 1 1 5EF40892
-P 1000 3250
-F 0 "#PWR0136" H 1000 3100 50  0001 C CNN
-F 1 "+3.3V" V 900 3300 50  0000 C CNN
-F 2 "" H 1000 3250 50  0000 C CNN
-F 3 "" H 1000 3250 50  0000 C CNN
-	1    1000 3250
-	1    0    0    -1
-$EndComp
-Wire Wire Line
-	1000 3250 1000 3400
+P 800 3250
+F 0 "#PWR0136" H 800 3100 50  0001 C CNN
+F 1 "+3.3V" V 700 3300 50  0000 C CNN
+F 2 "" H 800 3250 50  0000 C CNN
+F 3 "" H 800 3250 50  0000 C CNN
+	1    800  3250
+	1    0    0    -1
+$EndComp
+Wire Wire Line
+	800  3250 800  3400
 Wire Notes Line
 	10100 500  10100 750
@@
 Wire Wire Line
 	3650 850  3650 700
+Text GLabel 2000 3350 0    50   Input ~ 0
+GPIO3(SCL1)
+Text GLabel 2000 3250 0    50   Input ~ 0
+GPIO2(SDA1)
+$Comp
+L Device:R R13
+U 1 1 5FE27921
+P 2200 2800
+F 0 "R13" H 2270 2846 50  0000 L CNN
+F 1 "2k2" H 2270 2755 50  0000 L CNN
+F 2 "Resistor_SMD:R_0805_2012Metric" V 2130 2800 50  0001 C CNN
+F 3 "~" H 2200 2800 50  0001 C CNN
+	1    2200 2800
+	1    0    0    -1
+$EndComp
+$Comp
+L power:+3.3V #PWR012
+U 1 1 5FE47C2B
+P 2050 2550
+F 0 "#PWR012" H 2050 2400 50  0001 C CNN
+F 1 "+3.3V" V 1950 2600 50  0000 C CNN
+F 2 "" H 2050 2550 50  0000 C CNN
+F 3 "" H 2050 2550 50  0000 C CNN
+	1    2050 2550
+	1    0    0    -1
+$EndComp
+$Comp
+L power:+3.3V #PWR013
+U 1 1 5FE47C92
+P 2200 2550
+F 0 "#PWR013" H 2200 2400 50  0001 C CNN
+F 1 "+3.3V" V 2300 2600 50  0000 C CNN
+F 2 "" H 2200 2550 50  0000 C CNN
+F 3 "" H 2200 2550 50  0000 C CNN
+	1    2200 2550
+	1    0    0    -1
+$EndComp
+$Comp
+L Connector:Conn_01x04_Male J1
+U 1 1 5FD9DE9E
+P 2450 3250
+F 0 "J1" H 2423 3130 50  0000 R CNN
+F 1 "Conn_01x04_Male" H 2423 3221 50  0000 R CNN
+F 2 "Connector_PinHeader_2.54mm:PinHeader_1x04_P2.54mm_Horizontal" H 2450 3250 50  0001 C CNN
+F 3 "~" H 2450 3250 50  0001 C CNN
+	1    2450 3250
+	-1   0    0    1
+$EndComp
+$Comp
+L power:GND #PWR0106
+U 1 1 5FDAF246
+P 1350 3350
+F 0 "#PWR0106" H 1350 3100 50  0001 C CNN
+F 1 "GND" H 1350 3200 50  0000 C CNN
+F 2 "" H 1350 3350 50  0000 C CNN
+F 3 "" H 1350 3350 50  0000 C CNN
+	1    1350 3350
+	1    0    0    -1
+$EndComp
+$Comp
+L power:+3.3V #PWR0107
+U 1 1 5FDAF30D
+P 1350 2950
+F 0 "#PWR0107" H 1350 2800 50  0001 C CNN
+F 1 "+3.3V" V 1250 3000 50  0000 C CNN
+F 2 "" H 1350 2950 50  0000 C CNN
+F 3 "" H 1350 2950 50  0000 C CNN
+	1    1350 2950
+	1    0    0    -1
+$EndComp
+Wire Wire Line
+	2250 3150 1350 3150
+Wire Wire Line
+	1350 3150 1350 3350
+Wire Wire Line
+	1350 3050 1350 2950
+$Comp
+L Device:R R12
+U 1 1 5FE27881
+P 2050 2800
+F 0 "R12" H 1800 2850 50  0000 L CNN
+F 1 "2k2" H 1800 2750 50  0000 L CNN
+F 2 "Resistor_SMD:R_0805_2012Metric" V 1980 2800 50  0001 C CNN
+F 3 "~" H 2050 2800 50  0001 C CNN
+	1    2050 2800
+	1    0    0    -1
+$EndComp
+Wire Wire Line
+	2000 3350 2050 3350
+Wire Wire Line
+	2050 3350 2050 2950
+Connection ~ 2050 3350
+Wire Wire Line
+	2050 3350 2250 3350
+Wire Wire Line
+	2000 3250 2200 3250
+Wire Wire Line
+	1350 3050 2250 3050
+Wire Wire Line
+	2200 3250 2200 2950
+Connection ~ 2200 3250
+Wire Wire Line
+	2200 3250 2250 3250
+Wire Wire Line
+	2200 2650 2200 2550
+Wire Wire Line
+	2050 2650 2050 2550
 $EndSCHEMATC

Commit message: Change 26vias connector
Parts:
- J4: footprint Connector_PinSocket_2.54mm:PinSocket_2x13_P2.54mm_Vertical -> Connector_IDC:IDC-Header_2x13_P2.54mm_Vertical
Connections:
- net A2: now also J4.12 (Pin_12); no longer J4.11 (Pin_11)
- net A3: now also J4.6 (Pin_6); no longer J4.5 (Pin_5)
- net ADC0: now also J4.8 (Pin_8); no longer J4.7 (Pin_7)
- net ADC1: now also J4.10 (Pin_10); no longer J4.9 (Pin_9)
- net AMP1: now also J4.4 (Pin_4); no longer J4.3 (Pin_3)
- net AMP2: now also J4.14 (Pin_14); no longer J4.13 (Pin_13)
- net D0: now also J4.1 (Pin_1); no longer J4.2 (Pin_2)
- net D1: now also J4.23 (Pin_23); no longer J4.24 (Pin_24)
- net Echo0: now also J4.21 (Pin_21); no longer J4.22 (Pin_22)
- net Echo1: now also J4.5 (Pin_5); no longer J4.6 (Pin_6)
- net GND: now also J4.2 (Pin_2), J4.3 (Pin_3); no longer J4.1 (Pin_1), J4.4 (Pin_4)
- net L_TCRT: now also J4.13 (Pin_13); no longer J4.14 (Pin_14)
- net PWM1: now also J4.22 (Pin_22); no longer J4.21 (Pin_21)
- net PWM1N: now also J4.24 (Pin_24); no longer J4.23 (Pin_23)
- net PWM2: now also J4.26 (Pin_26); no longer J4.25 (Pin_25)
- net PWM2N: now also J4.25 (Pin_25); no longer J4.26 (Pin_26)
- net RXB: now also J4.20 (Pin_20); no longer J4.19 (Pin_19)
- net R_TCRT: now also J4.11 (Pin_11); no longer J4.12 (Pin_12)
- net TXB: now also J4.18 (Pin_18); no longer J4.17 (Pin_17)
- net Trig0: now also J4.19 (Pin_19); no longer J4.20 (Pin_20)
- net Trig1: now also J4.7 (Pin_7); no longer J4.8 (Pin_8)
Changed lines of the file:
@@
 L Connector_Generic:Conn_02x13_Odd_Even J4
 U 1 1 5EE18C86
-P 1400 1550
-F 0 "J4" H 1450 2367 50  0000 C CNN
-F 1 "Conn_02x13_Odd_Even" H 1450 2276 50  0000 C CNN
-F 2 "Connector_PinSocket_2.54mm:PinSocket_2x13_P2.54mm_Vertical" H 1400 1550 50  0001 C CNN
-F 3 "~" H 1400 1550 50  0001 C CNN
-	1    1400 1550
-	1    0    0    -1
+P 1500 1550
+F 0 "J4" H 1550 2367 50  0000 C CNN
+F 1 "Conn_02x13_Odd_Even" H 1550 2276 50  0000 C CNN
+F 2 "Connector_IDC:IDC-Header_2x13_P2.54mm_Vertical" H 1500 1550 50  0001 C CNN
+F 3 "~" H 1500 1550 50  0001 C CNN
+	1    1500 1550
+	-1   0    0    -1
 $EndComp
 Text GLabel 2150 950  2    50   Input ~ 0

Commit message: Added motor class
Other:
- note added: "HAT PARA CARRINHO AUTÔNOMO\nLIGAÇÃO CONFORME PLACA DE POTÊNCIA"
- note removed: "SHIELD EXP430FR2355 PARA CARRINHO AUTÔNOMO\nLIGAÇÃO CONFORME PLACA DE POTÊNCIA"
Changed lines of the file:
@@
 	800  4100 800  4200
 Text Notes 7000 6750 0    50   ~ 0
-SHIELD EXP430FR2355 PARA CARRINHO AUTÔNOMO\nLIGAÇÃO CONFORME PLACA DE POTÊNCIA
+HAT PARA CARRINHO AUTÔNOMO\nLIGAÇÃO CONFORME PLACA DE POTÊNCIA
 Text GLabel 3600 5500 2    50   Input ~ 0
 GPIO7(SPI1_CE_N)

Commit message: Change encoder gpio library
Parts:
- A1: symbol Charleslabs_Parts:ADS1115_ADC_Module -> hardware-rescue:ADS1115_ADC_Module-Charleslabs_Parts
Changed lines of the file:
@@
 EESchema Schematic File Version 4
-LIBS:hardware-cache
-EELAYER 26 0
+EELAYER 30 0
 EELAYER END
 $Descr A4 11693 8268
@@
 	2950 3250 2950 3450
 $Comp
-L Charleslabs_Parts:ADS1115_ADC_Module A1
+L hardware-rescue:ADS1115_ADC_Module-Charleslabs_Parts A1
 U 1 1 5F6D8D72
 P 2950 3950
