File: rasp/hardware/hardware.kicad_pcb (KiCad board)
At the start: 2 copper layers, 65 x 69 mm, 47 parts, among them J1 Conn_01x04_Male, J10 Conn_01x02_Male, J11 Conn_01x02_Male, J12 Conn_01x02_Male, J13 Conn_01x02_Male, J14 Conn_01x02_Male, J15 Conn_01x02_Male, J16 Conn_01x02_Male, J17 Conn_01x02_Male, J18 Conn_01x02_Male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

Commit message: Added boards
Routing:
- net A2: track 76.1 -> 76.3 mm, vias 4 -> 3
- net (no net): vias 4 -> 0
Changed lines of the file:
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@@
     (thickness 1.6)
     (drawings 68)
-    (tracks 551)
+    (tracks 545)
     (zones 0)
     (modules 47)
@@
     (visible_elements 7FFFFFFF)
     (pcbplotparams
-      (layerselection 0x00030_80000001)
+      (layerselection 0x01030_ffffffff)
       (usegerberextensions true)
       (usegerberattributes false)
@@
       (outputformat 1)
       (mirror false)
-      (drillshape 1)
+      (drillshape 0)
       (scaleselection 1)
-      (outputdirectory ""))
+      (outputdirectory "fabric/"))
   )
   (net 0 "")
@@
     (effects (font (size 2 1.7) (thickness 0.12)) (justify left))
   )
-  (via (at 200 152.54) (size 1.5) (drill 0.6) (layers F.Cu B.Cu) (net 0))
-  (via (at 200 83.52312) (size 1.5) (drill 0.6) (layers F.Cu B.Cu) (net 0))
-  (via (at 265.024 83.52312) (size 1.5) (drill 0.6) (layers F.Cu B.Cu) (net 0))
-  (via (at 265.024 152.54) (size 1.5) (drill 0.6) (layers F.Cu B.Cu) (net 0))
   (segment (start 252.832 116.726) (end 253.086 116.98) (width 0.635) (layer B.Cu) (net 1))
   (segment (start 250.038 116.726) (end 252.832 116.726) (width 0.635) (layer B.Cu) (net 1))
@@
   (segment (start 255.9562 104.98104) (end 257.01686 104.98104) (width 0.635) (layer F.Cu) (net 55))
   (segment (start 258.928 149.492) (end 258.928 107.47532) (width 0.635) (layer F.Cu) (net 55))
-  (via (at 248.85 137.05) (size 1.5) (drill 0.6) (layers F.Cu B.Cu) (net 56))
-  (segment (start 250.038 137.046) (end 248.854 137.046) (width 0.635) (layer B.Cu) (net 56))
-  (segment (start 248.854 137.046) (end 248.85 137.05) (width 0.635) (layer B.Cu) (net 56))
-  (segment (start 247.612119 129.859463) (end 246.002656 128.25) (width 0.635) (layer F.Cu) (net 56))
-  (segment (start 248.85 137.05) (end 247.61212 135.81212) (width 0.635) (layer F.Cu) (net 56))
-  (segment (start 247.61212 135.81212) (end 247.612119 129.859463) (width 0.635) (layer F.Cu) (net 56))
-  (segment (start 243.997343 128.25) (end 241.9 130.347343) (width 0.635) (layer F.Cu) (net 56))
-  (segment (start 246.002656 128.25) (end 243.997343 128.25) (width 0.635) (layer F.Cu) (net 56))
   (via (at 241.7 130.65) (size 1.5) (drill 0.6) (layers F.Cu B.Cu) (net 56))
-  (segment (start 241.9 130.347343) (end 241.9 130.45) (width 0.635) (layer F.Cu) (net 56))
-  (segment (start 241.9 130.45) (end 241.7 130.65) (width 0.635) (layer F.Cu) (net 56))
   (segment (start 241.7 131.71066) (end 243 133.01066) (width 0.635) (layer B.Cu) (net 56))
   (segment (start 241.7 130.65) (end 241.7 131.71066) (width 0.635) (layer B.Cu) (net 56))
@@
   (segment (start 229.468 143.4) (end 230.992 143.4) (width 0.635) (layer F.Cu) (net 56))
   (segment (start 227.544601 141.476601) (end 229.468 143.4) (width 0.635) (layer F.Cu) (net 56))
+  (segment (start 248.514 137.046) (end 250.038 137.046) (width 0.635) (layer F.Cu) (net 56))
+  (segment (start 241.9 130.45) (end 241.9 130.347343) (width 0.635) (layer F.Cu) (net 56))
+  (segment (start 247.612119 129.859463) (end 247.61212 136.14412) (width 0.635) (layer F.Cu) (net 56))
+  (segment (start 241.7 130.65) (end 241.9 130.45) (width 0.635) (layer F.Cu) (net 56))
+  (segment (start 241.9 130.347343) (end 243.997343 128.25) (width 0.635) (layer F.Cu) (net 56))
+  (segment (start 247.61212 136.14412) (end 248.514 137.046) (width 0.635) (layer F.Cu) (net 56))
+  (segment (start 243.997343 128.25) (end 246.002656 128.25) (width 0.635) (layer F.Cu) (net 56))
+  (segment (start 246.002656 128.25) (end 247.612119 129.859463) (width 0.635) (layer F.Cu) (net 56))
   (segment (start 238.7835 143.3175) (end 238.705 143.396) (width 0.635) (layer B.Cu) (net 58))
   (segment (start 238.7835 141.11) (end 238.7835 143.3175) (width 0.635) (layer B.Cu) (net 58))
